File: design/main_board/BLE.kicad_sch (KiCad schematic)
At the start: 6 parts, among them U201 RN4871

Commit message: Created esp32 footprint and symbol
Connections:
- net ~BLE_RST renamed ~{BLE_RST}
