File: design/main_board/camera.kicad_sch (KiCad schematic)
At the start: 18 parts

Commit message: Added new firmware hello world for ESP32-S3
Parts:
- removed C? (x2): 0.1uF, symbol Device:C
- removed C? (x3): 4.7uF, symbol Device:C
Connections:
- net AVDD_2V8 renamed VDD_2V8
- net VDD_2V8: no longer U?.4 (AVDD)
- net DVDD_1V5 renamed VDD_1V5
- net VDD_3V3 renamed VDD_5V
